File: Hardware/SparkFun_Audio_Player_Breakout_MY1690X-16S.kicad_pcb (KiCad board)
At the start: 4 copper layers, 25.4 x 25.4 mm, 74 parts, among them J1 3.5mm TRRS, J2 Conn_01x03, J3 Conn_01x02, J4 USB_C_Receptacle, J5 Conn_01x06, J6 microSD, Q1 BSS138, U2 MY1690X-16S

Commit message: Ordering instructions updated - panel/gerber v10c
-Material TG135-140
-Controlled Impedance: No
Other:
- board text added: "Controlled Impedance: No"
- board text added: "Material: TG135-140"
Changed lines of the file:
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@@
+		)
+	)
+	(gr_text "Controlled Impedance: No"
+		(at 188.95 153.653 0)
+		(layer "Eco1.User")
+		(effects
+			(font
+				(size 1.27 1.27)
+				(thickness 0.15)
+			)
+			(justify left bottom)
 		)
 	)
@@
 		(layer "Eco1.User")
 		(effects
+			(font
+				(size 1.27 1.27)
+				(thickness 0.15)
+			)
+			(justify left bottom)
+		)
+	)
+	(gr_text "Material: TG135-140"
+		(at 189.019 155.476 0)
+		(layer "Eco1.User")
+		(effects
